File: EDA/cube/cube.kicad_sch (KiCad schematic)
At the start: 17 parts, among them Q1 BC337, SW1 SW_Push, SW2 SW_Push, SW3 SW_Push, SW4 SW_Push, SW5 SW_Push, SW6 SW_SPDT, SW7 SW_SPDT

Commit message: [EDA] PCB v1.0-revA
Parts:
- added BT1: Battery_Cell, Connector_PinHeader_1.27mm:PinHeader_1x02_P1.27mm_Vertical, symbol Device:Battery_Cell
- LS1, SW1, SW2, SW3, SW4, SW5: footprint (none) -> Connector_PinHeader_1.27mm:PinHeader_1x02_P1.27mm_Vertical
- R1, R2, R3, R4, R5, R6: footprint (none) -> Resistor_THT:R_Axial_DIN0207_L6.3mm_D2.5mm_P7.62mm_Horizontal
- SW6, SW7: footprint (none) -> Button_Switch_THT:SW_Slide_1P2T_CK_OS102011MS2Q
- U1: footprint (none) -> custom:SD_AZDelivery
Connections:
- net GND: now also BT1.2 (-)
- net Vin: now reaches A1.30 (VIN), SW6.2 (B)
- net +5V: no longer names the net of SW6.1 (A)
- net +5V: now also BT1.1 (+)
- no-connect marks 1 -> 16
